Commit message: new laptop

File: description/robot_core.xacro (robot description, xacro)
@@ -21,4 +21,11 @@
     <link name="base_link">
     </link>
+    <joint name="base_footprint_joint" type="fixed">
+        <parent link="base_link"/>
+        <child link="base_footprint"/>
+        <origin xyz="0 0 0" rpy="0 0 0" />
+    </joint>
+    <link name="base_footprint">
+    </link>
     <joint name="chassis_joint" type="fixed">
         <parent link="base_link" />
@@ -41,5 +48,5 @@
         <collision>
             <geometry>
-                <cylinder length="0.04" radius="0.05" />
+                <sphere radius="0.05" />
             </geometry>
         </collision>
@@ -81,5 +88,5 @@
         <collision>
             <geometry>
-                <cylinder length="0.04" radius="0.05" />/> </geometry>
+                <sphere radius="0.05" />/> </geometry>
         </collision>
         <xacro:inertial_cylinder mass="0.1" length="0.05" radius="0.05">
